File: FlightController/FlightController.kicad_pcb (KiCad board)
At the start: 4 copper layers, 41.9 x 41.9 mm, 74 parts, among them J2 Conn_01x04_Pin, J3 SM08B-SRSS-TBLFSN, U1 AP2112K-3.3, U2 USBLC6-2SC6, U3 STM32F411CEUx, U4 ICM-42688-P, U5 BMP390, U6 TPS62933, U7 TPS2115ADRBR, Y1 25MHz_GND24

Commit message: Update PCB
Parts:
- moved R4 94.0 mm to (149.4, 106.8)
- moved C1 91.1 mm to (141.3, 104.3), turned to 90 degrees
- moved C21 89.5 mm to (131.7, 93.9), turned to 180 degrees
- moved U3 88.7 mm to (165.8, 93.5)
- moved C27 88.4 mm to (136.0, 93.9)
- moved U1 87.5 mm to (144.8, 106.3)
- moved U7 86.6 mm to (133.7, 97.0), turned to 90 degrees
- moved R12 86.5 mm to (136.2, 100.0)
- moved R1 83.7 mm to (142.3, 108.8)
- moved C28 83.5 mm to (135.3, 92.1)
- moved D2 82.5 mm to (149.5, 108.4), turned to 180 degrees
- moved C2 81.6 mm to (149.4, 104.9)
- moved J2 71.7 mm to (118.5, 95.8), turned to 90 degrees
- moved C11 69.6 mm to (160.5, 92.6), turned to 90 degrees
- moved Y1 66.4 mm to (157.6, 91.5), turned to -90 degrees
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Connections:
- U3 pad 42: /MCU/M1 -> /MCU/M4
- U3 pad 43: /MCU/M2 -> /MCU/M3
- U3 pad 45: /MCU/M3 -> /MCU/M2
- U3 pad 46: /MCU/M4 -> /MCU/M1
Routing:
- net IN2: track 0.00 -> 46.3 mm, vias 0 -> 2
- net +5V: track 0.00 -> 40.3 mm, vias 0 -> 2
- net +3.3V: track 0.00 -> 26.1 mm, vias 0 -> 2
- net /MCU/M2: track 0.00 -> 25.4 mm
- net /MCU/D+: track 0.00 -> 25.3 mm
- net /MCU/D-: track 0.00 -> 25.2 mm
- net /MCU/M1: track 0.00 -> 25.1 mm
- net /MCU/M3: track 0.00 -> 25.0 mm
- net /MCU/M4: track 0.00 -> 25.0 mm
- net GND: track 0.00 -> 20.2 mm, vias 0 -> 166
- net /IMU/MOSI: track 0.00 -> 12.9 mm
- net /IMU/MISO: track 0.00 -> 12.9 mm
- net /IMU/SCLK: track 0.00 -> 11.4 mm
- net IN1: track 24.8 -> 32.6 mm
- net Net-(U3-PH0): track 0.00 -> 7.77 mm
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- added copper zone on In1.Cu, net GND

Commit message: Final Update
Parts:
- removed BOOT1, NRST1: SW_Push, PCM_JLCPCB:SW_TS-1088-AR02016
- removed J2: Conn_01x04_Pin, Connector_PinHeader_1.00mm:PinHeader_1x04_P1.00mm_Vertical
- added G***: LOGO, LOGO, B.Cu at (150.8, 88.1)
- added J1: Conn_01x03_Pin, Connector_PinHeader_1.00mm:PinHeader_1x03_P1.00mm_Vertical, F.Cu at (161.4, 72.2)
- added JP1: SolderJumper_2_Open, Jumper:SolderJumper-2_P1.3mm_Open_Pad1.0x1.5mm, F.Cu at (171.2, 73.8)
- C4, C7, C8, C9: value 100nF X7R -> 0.1μF X7R
- TP1, TP2, TP3, TP4: moved to B.Cu
- Y1: footprint Crystal:Crystal_SMD_3225-4Pin_3.2x2.5mm_HandSoldering -> CRYSTAL-SMD_4P-L3.2-W2.5-BL:CRYSTAL-SMD_4P-L3.2-W2.5-BL
- moved TP1 116.7 mm to (155.2, 107.3), turned to 90 degrees
- moved TP2 111.6 mm to (151.2, 107.3), turned to 90 degrees
- moved C6 111.1 mm to (171.0, 102.5), turned to -90 degrees
- moved C7 108.9 mm to (170.9, 97.5), turned to 90 degrees
- moved C8 107.7 mm to (171.0, 90.2), turned to 90 degrees
- moved TP3 106.2 mm to (146.7, 107.3), turned to 90 degrees
- moved C5 101.8 mm to (169.0, 100.0)
- moved C9 101.3 mm to (162.9, 88.6), turned to 90 degrees
- moved TP4 101.2 mm to (142.3, 107.4), turned to 90 degrees
- moved C29 100.4 mm to (162.0, 104.7), turned to -90 degrees
- moved R16 97.4 mm to (158.9, 106.2), turned to 90 degrees
- moved R13 90.5 mm to (170.0, 106.9), turned to -90 degrees
- moved D1 86.2 mm to (158.2, 78.3), turned to 180 degrees
- moved R18 85.5 mm to (158.3, 76.8), turned to 180 degrees
- moved C3 85.1 mm to (160.8, 97.3), turned to -90 degrees
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Connections:
- net NRST renamed Net-(U3-NRST)
- U3 pad 26: STATUS_LED -> unconnected-(U3-PB13-Pad26)
- U3 pad 41: unconnected-(U3-PB5-Pad41) -> STATUS_LED
Routing:
- net +5V: track 40.3 -> 144.8 mm, vias 2 -> 5
- net +3.3V: track 26.1 -> 130.3 mm, vias 2 -> 10
- net +BATT: track 2.54 -> 87.9 mm, vias 0 -> 2
- net /MCU/CUR: track 0.00 -> 70.3 mm, vias 0 -> 2
- net /MCU/RX: track 0.00 -> 39.5 mm, vias 0 -> 1
- net /MCU/TX: track 0.00 -> 34.2 mm, vias 0 -> 1
- net /IMU/INT1_IMU: track 0.00 -> 26.8 mm, vias 0 -> 2
- net /MCU/SWDIO: track 0.00 -> 25.4 mm, vias 0 -> 2
- net /MCU/SWCLK: track 0.00 -> 25.0 mm, vias 0 -> 2
- net BOOT0: track 0.00 -> 23.6 mm, vias 0 -> 3
- net Net-(U3-NRST): track 0.00 -> 19.6 mm
- net /IMU/CS_BMP: track 0.00 -> 17.7 mm, vias 0 -> 2
- net STATUS_LED: track 0.00 -> 17.2 mm, vias 0 -> 2
- net /IMU/CS_IMU: track 3.45 -> 19.4 mm, vias 0 -> 2
- net Net-(U3-PB0): track 0.00 -> 14.2 mm, vias 0 -> 2
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- added copper zone on B.Cu, net GND
- added copper zone on F.Cu, net GND
- added copper zone on In2.Cu, net GND
Other:
- board size 41.9 x 41.9 mm -> 45 x 45 mm
- board text added: "27/09/2026"
- board text added: "3.3V"
- board text added: "BOOT0"
- board text added: "JLCJLCJLCJLC"
- board text added: "QuadFlyController V 1.0 M. Alejandro Sanchez R."
